File: Hardware/CPU/ScreenHat/ScreenHat/_autosave-ScreenHat.kicad_pcb (KiCad board)
At the start: 2 copper layers, 156.5 x 63 mm, 48 parts, among them J10 Conn_02x01, J11 Conn_02x01, J8 Conn_02x01, J9 Conn_02x01, SW1 Push_Button, SW2 Push_Button, SW3 Push_Button, SW4 Push_Button, SW5 Push_Button, SW6 Push_Button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

Commit message: finished ScreenHat Schematics
Parts:
- J10, J11, J8: moved to B.Cu
- moved U3 214.1 mm to (199.8, 34.7)
- moved J8 184.9 mm to (245.5, 3.00)
- moved J11 164.0 mm to (245.5, 60.5)
- moved J10 27.2 mm to (97.0, 60.5)
- moved J9 0.27 mm to (97.0, 3.00)
Other:
- board size 156.5 x 63 mm -> 157 x 63.5 mm
