File: Hardware/CPU/ScreenHat/ScreenHat/ScreenHat.kicad_pcb (KiCad board)
At the start: 2 copper layers, 156.5 x 63 mm, 48 parts, among them J10 Conn_02x01, J11 Conn_02x01, J8 Conn_02x01, J9 Conn_02x01, SW1 Push_Button, SW2 Push_Button, SW3 Push_Button, SW4 Push_Button, SW5 Push_Button, SW6 Push_Button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

Commit message: started designing ScreenHat Board
Parts:
- added Q2: BC417, PCM_Package_TO_SOT_SMD_AKL:SOT-23, F.Cu at (152.0, 10.0)
- C1, C2, C3, C4, C5, C6, C7: footprint Capacitor_THT:C_Disc_D3.0mm_W2.0mm_P2.50mm -> Capacitor_SMD:C_0805_2012Metric_Pad1.18x1.45mm_HandSolder
- J10, J11, J8, JP1, JP2, JP3, JP4, JP5, JP6: moved to B.Cu
- R2: value R -> 4.7k; footprint PCM_Resistor_SMD_AKL:R_0805_2012Metric_Pad1.15x1.40mm_HandSolder -> PCM_Resistor_SMD_AKL:R_0805_2012Metric
- moved C4 271.6 mm to (247.5, 24.5)
- moved C1 258.2 mm to (232.5, 9.00)
- moved C7 256.5 mm to (236.0, 56.0), turned to 180 degrees
- moved C5 256.3 mm to (234.0, 38.0)
- moved C3 256.2 mm to (232.5, 24.5)
- moved C2 239.8 mm to (216.5, 24.5)
- moved C6 238.9 mm to (218.5, 53.5)
- moved R8 230.3 mm to (247.5, 26.5)
- moved R1 217.6 mm to (232.5, 11.0)
- moved LED2 217.2 mm to (241.6, 46.5)
- moved R12 215.8 mm to (244.0, 56.6), turned to 90 degrees
- moved R7 215.0 mm to (232.5, 26.5)
- moved LED1 214.9 mm to (241.6, 56.0)
- moved R9 214.8 mm to (234.0, 40.0)
- moved R11 214.5 mm to (236.0, 58.0), turned to 180 degrees
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Connections:
- R2 pad 1: Net-(U1-P3) -> +3.3V
- R2 pad 2: Net-(Q1-PadB) -> Net-(Q2-B)
- U1 pad 7: Net-(U1-P3) -> Net-(Q2-B)
Routing:
- net GND: track 0.00 -> 594.3 mm
- net +3.3V: track 0.00 -> 310.2 mm, vias 0 -> 1
- net /SDA: track 0.00 -> 133.7 mm, vias 0 -> 3
- net /SCL: track 0.00 -> 133.6 mm, vias 0 -> 3
- net Net-(Q2-B): track 0.00 -> 31.6 mm
- net Net-(U1-P0): track 0.00 -> 30.7 mm
- net /LeftButton: track 0.00 -> 30.3 mm, vias 0 -> 2
- net Net-(U1-P1): track 0.00 -> 30.2 mm
- net Net-(U1-P2): track 0.00 -> 29.7 mm
- net Net-(U1-P7): track 0.00 -> 27.7 mm
- net /RunStopLED: track 0.00 -> 24.6 mm
- net Net-(U1-P6): track 0.00 -> 24.6 mm
- net Net-(U1-P5): track 0.00 -> 21.4 mm
- net Net-(U1-P4): track 0.00 -> 16.1 mm
- net Net-(JP1-A): track 0.00 -> 14.1 mm, vias 0 -> 1
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Other:
- board size 156.5 x 63 mm -> 157 x 63.5 mm
